File: hardware/magnetic-chess-board/magnetic-chess-board.kicad_pcb (KiCad board)
At the start: 2 copper layers, 207.1 x 188 mm, 132 parts, among them J1 OLED_128x64, SW1 SW_Reed, SW10 SW_Reed, SW11 SW_Reed, SW12 SW_Reed, SW13 SW_Reed, SW14 SW_Reed, SW15 SW_Reed, SW16 SW_Reed, SW17 SW_Reed, SW18 SW_Reed, SW19 SW_Reed, SW2 SW_Reed, SW20 SW_Reed, SW21 SW_Reed, SW22 SW_Reed, SW23 SW_Reed, SW24 SW_Reed, SW25 SW_Reed, SW26 SW_Reed, SW27 SW_Reed, SW28 SW_Reed, SW29 SW_Reed, SW3 SW_Reed, SW30 SW_Reed, SW31 SW_Reed, SW32 SW_Reed, SW33 SW_Reed, SW34 SW_Reed, SW35 SW_Reed, SW36 SW_Reed, SW37 SW_Reed, SW38 SW_Reed, SW39 SW_Reed, SW4 SW_Reed, SW40 SW_Reed, SW41 SW_Reed, SW42 SW_Reed, SW43 SW_Reed, SW44 SW_Reed, SW45 SW_Reed, SW46 SW_Reed, SW47 SW_Reed, SW48 SW_Reed, SW49 SW_Reed, SW5 SW_Reed, SW50 SW_Reed, SW51 SW_Reed, SW52 SW_Reed, SW53 SW_Reed, SW54 SW_Reed, SW55 SW_Reed, SW56 SW_Reed, SW57 SW_Reed, SW58 SW_Reed, SW59 SW_Reed, SW6 SW_Reed, SW60 SW_Reed, SW61 SW_Reed, SW62 SW_Reed, SW63 SW_Reed, SW64 SW_Reed, SW7 SW_Reed, SW8 SW_Reed, SW9 SW_Reed

Commit message: Refactor code structure for improved readability and maintainability
Parts:
- added REF**: MountingHole_3.2mm_M3, MountingHole:MountingHole_3.2mm_M3, F.Cu at (303.6, 234.0)
- added REF**: MountingHole_3.2mm_M3, MountingHole:MountingHole_3.2mm_M3, F.Cu at (116.5, 66.0)
- added REF** (x2): MountingHole_3.2mm_M3, MountingHole:MountingHole_3.2mm_M3, F.Cu at (116.5, 234.0)
- added REF**: MountingHole_3.2mm_M3, MountingHole:MountingHole_3.2mm_M3, F.Cu at (303.6, 66.0)
