File: magnetic-chess-board/magnetic-chess-board.kicad_pcb (KiCad board)
At the start: 2 copper layers, 207.1 x 188 mm, 132 parts, among them J1 OLED_128x64, SW1 SW_Reed, SW10 SW_Reed, SW11 SW_Reed, SW12 SW_Reed, SW13 SW_Reed, SW14 SW_Reed, SW15 SW_Reed, SW16 SW_Reed, SW17 SW_Reed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

Commit message: Key
Parts:
- S1, S2: footprint ScottoKeebs_Choc:Choc_V2 -> KiSwitch_Hotswap_Kalih:SW_Hotswap_Kailh_Choc_V1
