File: magnetic-chess-board/magnetic-chess-board.kicad_sch (KiCad schematic)
At the start: 132 parts, among them J1 OLED_128x64, SW1 SW_Reed, SW10 SW_Reed, SW11 SW_Reed, SW12 SW_Reed, SW13 SW_Reed, SW14 SW_Reed, SW15 SW_Reed, SW16 SW_Reed, SW17 SW_Reed, SW18 SW_Reed, SW19 SW_Reed, SW2 SW_Reed, SW20 SW_Reed, SW21 SW_Reed, SW22 SW_Reed, SW23 SW_Reed, SW24 SW_Reed, SW25 SW_Reed, SW26 SW_Reed, SW27 SW_Reed, SW28 SW_Reed, SW29 SW_Reed, SW3 SW_Reed, SW30 SW_Reed, SW31 SW_Reed, SW32 SW_Reed, SW33 SW_Reed, SW34 SW_Reed, SW35 SW_Reed, SW36 SW_Reed, SW37 SW_Reed, SW38 SW_Reed, SW39 SW_Reed, SW4 SW_Reed, SW40 SW_Reed, SW41 SW_Reed, SW42 SW_Reed, SW43 SW_Reed, SW44 SW_Reed, SW45 SW_Reed, SW46 SW_Reed, SW47 SW_Reed, SW48 SW_Reed, SW49 SW_Reed, SW5 SW_Reed, SW50 SW_Reed, SW51 SW_Reed, SW52 SW_Reed, SW53 SW_Reed, SW54 SW_Reed, SW55 SW_Reed, SW56 SW_Reed, SW57 SW_Reed, SW58 SW_Reed, SW59 SW_Reed, SW6 SW_Reed, SW60 SW_Reed, SW61 SW_Reed, SW62 SW_Reed, SW63 SW_Reed, SW64 SW_Reed, SW7 SW_Reed, SW8 SW_Reed, SW9 SW_Reed

Commit message: Key
Parts:
- S1, S2: footprint ScottoKeebs_Choc:Choc_V2 -> KiSwitch_Hotswap_Kalih:SW_Hotswap_Kailh_Choc_V1
Changed lines of the file:
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@@
 			)
 		)
-		(property "Footprint" "ScottoKeebs_Choc:Choc_V2"
+		(property "Footprint" "KiSwitch_Hotswap_Kalih:SW_Hotswap_Kailh_Choc_V1"
 			(at 379.73 82.55 0)
 			(hide yes)
@@
 			)
 		)
-		(property "Footprint" "ScottoKeebs_Choc:Choc_V2"
+		(property "Footprint" "KiSwitch_Hotswap_Kalih:SW_Hotswap_Kailh_Choc_V1"
 			(at 379.73 88.9 0)
 			(hide yes)
